File: hardware/vl53l0_breakout/vl53l0_breakout.kicad_sch (KiCad schematic)
At the start: 15 parts, among them J1 Conn_01x06, U1 VL53L0CXV0DH1

Commit message: routing
Parts:
- added H1, H2: MountingHole_Pad, MountingHole:MountingHole_2.2mm_M2_ISO7380_Pad, symbol Mechanical:MountingHole_Pad
- C3: footprint Capacitor_SMD:C_0402_1005Metric -> Capacitor_SMD:C_0603_1608Metric; JLCPCB C15525 -> C15850
Connections:
- net GND: now also H1.1, H2.1
