File: hardware/vl53l0_breakout/vl53l0_breakout.kicad_pcb (KiCad board)
At the start: 2 copper layers, 15 parts, among them J1 Conn_01x06, U1 VL53L0CXV0DH1

Commit message: routing
Parts:
- added H1: MountingHole_Pad, MountingHole:MountingHole_2.2mm_M2_ISO7380_Pad, F.Cu at (151.0, 67.5)
- added H2: MountingHole_Pad, MountingHole:MountingHole_2.2mm_M2_ISO7380_Pad, F.Cu at (151.0, 80.5)
- C3: footprint Capacitor_SMD:C_0402_1005Metric -> Capacitor_SMD:C_0603_1608Metric
- moved R7 10.1 mm to (147.5, 80.1), turned to -90 degrees
- moved R1 6.09 mm to (147.5, 78.1), turned to 90 degrees
- moved D2 5.90 mm to (147.3, 68.9), turned to 90 degrees
- moved R4 5.08 mm to (145.7, 75.3)
- moved R8 5.03 mm to (147.3, 72.5)
- moved C3 4.74 mm to (145.7, 68.9)
- moved J1 4.72 mm to (143.0, 67.7)
- moved R5 4.70 mm to (145.7, 77.8)
- moved R3 4.64 mm to (145.7, 72.7)
- moved C2 4.55 mm to (151.3, 70.5), turned to 180 degrees
- moved C1 4.51 mm to (149.3, 70.5)
- moved R9 4.40 mm to (147.3, 74.8)
- moved R6 4.34 mm to (145.7, 80.4)
- moved R2 4.29 mm to (146.5, 66.8)
- moved U1 4.00 mm to (150.0, 74.0)
Routing:
- net +3.3V: track 0.00 -> 33.3 mm, vias 0 -> 3
- net /TOF_XSHUT: track 0.00 -> 8.01 mm
- net GND: track 0.00 -> 7.09 mm, vias 0 -> 4
- net /TOF_GPIO1: track 0.00 -> 4.33 mm
- net /TOF_I2C_SDA: track 0.00 -> 3.84 mm
- net /TOF_I2C_SCL: track 0.00 -> 3.13 mm
- net /XSHUT: track 0.00 -> 2.24 mm
- net /I2C_SDA: track 0.00 -> 2.24 mm
- net /I2C_SCL: track 0.00 -> 2.24 mm
- net /GPIO1: track 0.00 -> 2.24 mm
- net /LEDK: track 0.00 -> 1.43 mm
- added copper zone on B.Cu, net GND
Other:
- board outline added: 12 x 17 mm
- board text added: "3.3V"
- board text added: "GND"
- board text added: "GPIO1"
- board text added: "SCL"
- board text added: "SDA"
- board text added: "VL53L0 CXV0DH1"
- board text added: "XST"

Commit message: modif + gerber
Parts:
- moved H1 0.50 mm to (151.0, 67.0)
- moved H2 0.50 mm to (151.0, 81.0)
Other:
- board size 12 x 17 mm -> 12 x 18 mm
Changed lines of the file:
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@@
 			(usegerberattributes yes)
 			(usegerberadvancedattributes yes)
-			(creategerberjobfile yes)
+			(creategerberjobfile no)
 			(dashed_line_dash_ratio 12.000000)
 			(dashed_line_gap_ratio 3.000000)
@@
 			(outputformat 1)
 			(mirror no)
-			(drillshape 1)
+			(drillshape 0)
 			(scaleselection 1)
-			(outputdirectory "")
+			(outputdirectory "../vl53l0_gerber/")
 		)
 	)
@@
 	(footprint "MountingHole:MountingHole_2.2mm_M2_ISO7380_Pad"
 		(layer "F.Cu")
-		(at 151 67.5)
+		(at 151 67)
 		(descr "Mounting Hole 2.2mm, M2, generated by kicad-footprint-generator mountinghole.py")
 		(tags "mountinghole M2 ISO7380")
@@
 	(footprint "MountingHole:MountingHole_2.2mm_M2_ISO7380_Pad"
 		(layer "F.Cu")
-		(at 151 80.5)
+		(at 151 81)
 		(descr "Mounting Hole 2.2mm, M2, generated by kicad-footprint-generator mountinghole.py")
 		(tags "mountinghole M2 ISO7380")
@@
 	)
 	(gr_line
-		(start 142.4 65.5)
-		(end 151 65.5)
+		(start 142.4 65)
+		(end 151 65)
 		(stroke
 			(width 0.05)
@@
 	)
 	(gr_arc
-		(start 141 66.9)
-		(mid 141.410051 65.910051)
-		(end 142.4 65.5)
+		(start 141 66.4)
+		(mid 141.410051 65.410051)
+		(end 142.4 65)
 		(stroke
 			(width 0.05)
@@
 	)
 	(gr_line
-		(start 151 82.5)
-		(end 142.2 82.5)
+		(start 151 83)
+		(end 142.2 83)
 		(stroke
 			(width 0.05)
@@
 	)
 	(gr_arc
-		(start 153 80.5)
-		(mid 152.414214 81.914214)
-		(end 151 82.5)
+		(start 153 81)
+		(mid 152.414214 82.414214)
+		(end 151 83)
 		(stroke
 			(width 0.05)
@@
 	)
 	(gr_arc
-		(start 142.2 82.5)
-		(mid 141.351472 82.148528)
-		(end 141 81.3)
+		(start 142.2 83)
+		(mid 141.351472 82.648528)
+		(end 141 81.8)
 		(stroke
 			(width 0.05)
@@
 	)
 	(gr_line
-		(start 153 67.5)
-		(end 153 80.5)
+		(start 153 67)
+		(end 153 81)
 		(stroke
 			(width 0.05)
@@
 	)
 	(gr_line
-		(start 141 81.3)
-		(end 141 66.9)
+		(start 141 81.8)
+		(end 141 66.4)
 		(stroke
 			(width 0.05)
@@
 	)
 	(gr_arc
-		(start 151 65.5)
-		(mid 152.414214 66.085786)
-		(end 153 67.5)
+		(start 151 65)
+		(mid 152.414214 65.585786)
+		(end 153 67)
 		(stroke
 			(width 0.05)
@@
 		(layer "User.2")
 		(pts
-			(xy 151 80.5) (xy 151 67.5)
+			(xy 151 81) (xy 151 67)
 		)
 		(height 5)
@@
 			(keep_text_aligned yes)
 		)
-		(gr_text "13"
+		(gr_text "14"
 			(at 154.85 74 90)
 			(layer "User.2")
@@
 		(layer "User.2")
 		(pts
-			(xy 151 65.5) (xy 151 82.5)
+			(xy 151 65) (xy 151 83)
 		)
 		(height 8)
@@
 			(keep_text_aligned yes)
 		)
-		(gr_text "17"
+		(gr_text "18"
 			(at 157.85 74 90)
 			(layer "User.2")
@@
 		(polygon
 			(pts
-				(xy 140 65) (xy 154 65) (xy 154 83) (xy 140 83)
+				(xy 140 64.5) (xy 154 64.5) (xy 154 83.5) (xy 140 83.5)
 			)
 		)
